File: Electronic/DisplayTTL/DisplayTTL.kicad_pcb (KiCad board)
At the start: 2 copper layers, 55 x 55 mm, 26 parts, among them J1 Conn_01x05, J10 Conn_01x03, J11 Conn_01x10, J12 Conn_01x02, J2 Conn_01x04, J3 Conn_01x04, J4 TC2050, J5 Conn_01x02, J6 Conn_01x04, J7 Conn_01x04, J8 Conn_01x02, J9 Conn_01x03, U1 ATA6563-GAQW1, U2 MCP2518FDT-E/SL, U3 ES8388, U4 Core1106, U5 ESP32-P4-MODULE-32MB, U6 TPS61169DCKR

Commit message: Add RV1106 RGB666 pinout doc: bus mapping, pin allocation, GPIO recovery plan
Schematic:
- Wire most of the gpios,
- Button for boot / reset
- DIsplay schematic done
- Wip I2S codec wiring on ESP32-P4 side
- Single Pair Ethernet T1S
- I2C ADC with 4 input
- Core1106 / ESP32-P4 wiring mostly done

WIP PCB layout / schematic.

Docs:
- Add Pico Pi schematic (use the Core1106 module)
- Add Makerworld url for stick and stick position
Parts:
- removed J10: Conn_01x03, Connector_PinSocket_2.54mm:PinSocket_1x03_P2.54mm_Vertical
- removed the J4 at (70.6, 35.9)
- removed the J8 at (51.7, 68.3)
- added C1: 0.1uF, Capacitor_SMD:C_0201_0603Metric, F.Cu at (78.3, 114.3)
- added C1: 0.1uF, Capacitor_SMD:C_0201_0603Metric, F.Cu at (106.1, 48.2)
- added C10: 0.1uF, Capacitor_SMD:C_0201_0603Metric, F.Cu at (83.0, 111.0)
- added C10: 0.1uF, Capacitor_SMD:C_0201_0603Metric, F.Cu at (108.5, 51.7)
- added C11: 10pF, Capacitor_SMD:C_0201_0603Metric, F.Cu at (76.3, 103.9)
- added C11: 0.1uF, Capacitor_SMD:C_0201_0603Metric, F.Cu at (108.5, 53.4)
- added C12: 0.1uF, Capacitor_SMD:C_0402_1005Metric, F.Cu at (113.7, 18.4)
- added C12: 10nF, Capacitor_SMD:C_0201_0603Metric, F.Cu at (80.6, 102.6)
- added C13: 10pF, Capacitor_SMD:C_0201_0603Metric, F.Cu at (108.5, 55.2)
- added C13: 10nF, Capacitor_SMD:C_0201_0603Metric, F.Cu at (85.2, 102.0)
- added C14: 10nF, Capacitor_SMD:C_0201_0603Metric, F.Cu at (78.4, 109.0)
- added C14: 10nF, Capacitor_SMD:C_0201_0603Metric, F.Cu at (111.0, 48.2)
- added C15: 10nF, Capacitor_SMD:C_0201_0603Metric, F.Cu at (84.0, 111.0)
- added C15: 10nF, Capacitor_SMD:C_0201_0603Metric, F.Cu at (111.0, 49.9)
- added C16: 10nF, Capacitor_SMD:C_0201_0603Metric, F.Cu at (111.0, 51.7)
- added C16: 10uF, Capacitor_SMD:C_0402_1005Metric, F.Cu at (79.1, 102.3)
- added C17: 10nF, Capacitor_SMD:C_0201_0603Metric, F.Cu at (111.0, 53.4)
- added C17: 10uF, Capacitor_SMD:C_0402_1005Metric, F.Cu at (85.4, 102.9)
- added C18: 0.1uF, Capacitor_SMD:C_0402_1005Metric, F.Cu at (113.7, 20.4)
- added C18: 10uF, Capacitor_SMD:C_0402_1005Metric, F.Cu at (77.0, 109.3)
- added C19: 10uF, Capacitor_SMD:C_0402_1005Metric, F.Cu at (83.9, 112.1)
- added C19: 10uF, Capacitor_SMD:C_0402_1005Metric, F.Cu at (126.9, 50.3)
- added C2: 0.1uF, Capacitor_SMD:C_0201_0603Metric, F.Cu at (106.1, 49.9)
- added C2: 0.1uF, Capacitor_SMD:C_0201_0603Metric, F.Cu at (82.9, 113.9)
- added C20: 10uF, Capacitor_SMD:C_0402_1005Metric, F.Cu at (126.9, 52.2)
- added C21: 10uF, Capacitor_SMD:C_0402_1005Metric, F.Cu at (126.9, 54.2)
- added C22: 10uF, Capacitor_SMD:C_0402_1005Metric, F.Cu at (126.9, 56.2)
- added C23: 0.1uF, Capacitor_SMD:C_0402_1005Metric, F.Cu at (140.2, 89.1)
- added C24: 0.1uF, Capacitor_SMD:C_0402_1005Metric, F.Cu at (140.2, 91.1)
- added C25: 0.1uF, Capacitor_SMD:C_0402_1005Metric, F.Cu at (135.6, 78.3)
- added C26: 0.1uF, Capacitor_SMD:C_0402_1005Metric, F.Cu at (113.7, 24.3)
- added C27: 0.1uF, Capacitor_SMD:C_0402_1005Metric, F.Cu at (113.7, 26.3)
- added C3: 0.1uF, Capacitor_SMD:C_0201_0603Metric, F.Cu at (88.3, 112.9)
- added C3: 0.1uF, Capacitor_SMD:C_0201_0603Metric, F.Cu at (106.1, 51.7)
- added C37: 0.1uF, Capacitor_SMD:C_0402_1005Metric, F.Cu at (108.8, 16.4)
- added C38: 1uF, Capacitor_SMD:C_0402_1005Metric, F.Cu at (108.8, 18.4)
- added C39: 1uF, Capacitor_SMD:C_0402_1005Metric, F.Cu at (108.8, 20.4)
- added C4: 0.1uF, Capacitor_SMD:C_0402_1005Metric, F.Cu at (113.7, 16.4)
- added C4: 0.1uF, Capacitor_SMD:C_0201_0603Metric, F.Cu at (78.0, 113.0)
- added C5: 4.7uF, Capacitor_SMD:C_0402_1005Metric, F.Cu at (82.9, 102.2)
- added C5: 0.1uF, Capacitor_SMD:C_0201_0603Metric, F.Cu at (106.1, 53.4)
- added C6: 4.7uF, Capacitor_SMD:C_0402_1005Metric, F.Cu at (126.9, 48.3)
- added C6: 0.1uF, Capacitor_SMD:C_0402_1005Metric, F.Cu at (75.9, 109.3)
- added C7: 0.1uF, Capacitor_SMD:C_0201_0603Metric, F.Cu at (106.1, 55.2)
- added C7: 0.1uF, Capacitor_SMD:C_0201_0603Metric, F.Cu at (84.0, 110.2)
- added C8: 0.1uF, Capacitor_SMD:C_0201_0603Metric, F.Cu at (108.5, 48.2)
- added C8: 10pF, Capacitor_SMD:C_0201_0603Metric, F.Cu at (78.8, 106.0)
- added C9: 0.1uF, Capacitor_SMD:C_0201_0603Metric, F.Cu at (80.3, 101.3)
- added C9: 10pF, Capacitor_SMD:C_0201_0603Metric, F.Cu at (108.5, 49.9)
- added D1: B5819WS_C6067464, lcsc:SOD-323F_L1.7-W1.3-LS2.5-R-RD-1, F.Cu at (152.0, 82.5)
- added D2: MBR0540, Diode_SMD:D_SOD-123, F.Cu at (133.3, 46.5)
- added JP1: Jumper_2_Open, Jumper:SolderJumper-2_P1.3mm_Open_RoundedPad1.0x1.5mm, F.Cu at (88.2, 110.7)
- added JP1: Jumper_2_Open, Jumper:SolderJumper-2_P1.3mm_Open_RoundedPad1.0x1.5mm, F.Cu at (123.3, 49.1)
- added JP2: Jumper_2_Open, Jumper:SolderJumper-2_P1.3mm_Open_RoundedPad1.0x1.5mm, F.Cu at (78.2, 110.9)
- added JP2: Jumper_2_Open, Jumper:SolderJumper-2_P1.3mm_Open_RoundedPad1.0x1.5mm, F.Cu at (123.3, 52.6)
- added L1: DLW32MH201XK2L, lcsc:FILTER-SMD_4P-L3.2-W2.5-BL_DLW32SH510XK2L, F.Cu at (80.7, 112.4)
- added L2: BLM18KG331SN1D, lcsc:L0603, F.Cu at (78.8, 103.5)
- added L3: YNR4010-6R8M, lcsc:IND-SMD_L4.0-W4.0, F.Cu at (133.3, 42.2)
- added R1: 100K, Resistor_SMD:R_0201_0603Metric, F.Cu at (87.5, 112.9)
- added R1: 100K, Resistor_SMD:R_0201_0603Metric, F.Cu at (111.0, 55.2)
- added R13: 1R 1%, Resistor_SMD:R_0201_0603Metric, F.Cu at (106.1, 16.3)
- added R14: 10K, Resistor_SMD:R_0201_0603Metric, F.Cu at (106.1, 18.1)
- added R15: 10K, Resistor_SMD:R_0201_0603Metric, F.Cu at (106.1, 19.8)
- added R16: 100R, Resistor_SMD:R_0201_0603Metric, F.Cu at (106.1, 21.6)
- added R2: 49.9R, Resistor_SMD:R_0201_0603Metric, F.Cu at (113.4, 48.2)
- added R2: 49.9R, Resistor_SMD:R_0201_0603Metric, F.Cu at (86.5, 113.5)
- added R3: 49.9R, Resistor_SMD:R_0201_0603Metric, F.Cu at (113.4, 49.9)
- added R3: 49.9R, Resistor_SMD:R_0201_0603Metric, F.Cu at (76.3, 112.4)
- added R4: 100K, Resistor_SMD:R_0201_0603Metric, F.Cu at (113.4, 51.7)
- added R4: 100K, Resistor_SMD:R_0201_0603Metric, F.Cu at (78.8, 113.1)
- added R5: 12.4K 1%, Resistor_SMD:R_0201_0603Metric, F.Cu at (79.2, 104.6)
- added R5: 12.4K 1%, Resistor_SMD:R_0201_0603Metric, F.Cu at (113.4, 53.4)
- added R6: 10K, Resistor_SMD:R_0201_0603Metric, F.Cu at (87.8, 108.8)
- added R6: 10K, Resistor_SMD:R_0201_0603Metric, F.Cu at (113.4, 55.2)
- added SW1: SH-1808SN-250GF, lcsc:SW-SMD_4P-L4.2-W3.4-P2.15-LS5.2, F.Cu at (117.9, 49.6)
- added SW2: SH-1808SN-250GF, lcsc:SW-SMD_4P-L4.2-W3.4-P2.15-LS5.2, F.Cu at (117.9, 54.3)
- added TP1: TestPoint, TestPoint:TestPoint_Pad_D1.5mm, F.Cu at (124.3, 32.2)
- added TP12: TestPoint, TestPoint:TestPoint_Pad_D1.5mm, F.Cu at (148.1, 83.0)
- added TP13: TestPoint, TestPoint:TestPoint_Pad_D1.5mm, F.Cu at (148.1, 86.6)
- added TP14: TestPoint, TestPoint:TestPoint_Pad_D1.5mm, F.Cu at (132.1, 32.2)
- added TP15: TestPoint, TestPoint:TestPoint_Pad_D1.5mm, F.Cu at (132.1, 35.7)
- added TP2: TestPoint, TestPoint:TestPoint_Pad_D1.5mm, F.Cu at (124.3, 35.7)
- added TP3: TestPoint, TestPoint:TestPoint_Pad_D1.5mm, F.Cu at (76.3, 113.8)
- added TP3: TestPoint, TestPoint:TestPoint_Pad_D1.5mm, F.Cu at (124.3, 39.3)
- added TP4: TestPoint, TestPoint:TestPoint_Pad_D1.5mm, F.Cu at (124.3, 42.8)
- added TP4: TestPoint, TestPoint:TestPoint_Pad_D1.5mm, F.Cu at (84.8, 113.8)
- added U1: LAN8651B1-E/LMX, lcsc:VQFN-32_L5.0-W5.0-P0.50-TL-EP3.6, F.Cu at (83.2, 106.6)
- added U11: ES8388, Package_DFN_QFN:QFN-28-1EP_4x4mm_P0.45mm_EP2.6x2.6mm, F.Cu at (137.4, 33.5)
- added U2: AVRH10C221KT1R5YA8, lcsc:R0402, F.Cu at (87.8, 114.2)
- added U6: ESD5451N_C5261080, lcsc:DFN1006-2L-BI, F.Cu at (143.0, 89.1)
- added U7: ESD5451N_C5261080, lcsc:DFN1006-2L-BI, F.Cu at (143.0, 91.0)
- added U8: ADS1115IDGSR, lcsc:MSOP-10_L3.0-W3.0-P0.50-LS5.0-BL, F.Cu at (141.1, 84.7)
- added X1: ABM10-25.000MHZ-D30-T3, lcsc:CRYSTAL-SMD_4P-L2.5-W2.0-BL-B, F.Cu at (77.0, 106.5)
- J3: value Conn_01x04 -> Conn_01x02; footprint Connector_PinSocket_2.54mm:PinSocket_1x04_P2.54mm_Vertical -> Connector_PinSocket_2.54mm:PinSocket_1x02_P2.54mm_Vertical
- J9: value Conn_01x03 -> TC2050; footprint Connector_PinSocket_2.54mm:PinSocket_1x03_P2.54mm_Vertical -> Connector:Tag-Connect_TC2050-IDC-NL_2x05_P1.27mm_Vertical
- U3: value ES8388 -> AVRH10C221KT1R5YA8; footprint Package_DFN_QFN:QFN-28-1EP_4x4mm_P0.45mm_EP2.6x2.6mm -> lcsc:R0402
- moved J3 96.4 mm to (136.4, 83.6)
- moved J9 43.8 mm to (140.0, 74.5)
- moved U3 35.2 mm to (75.9, 111.1), turned to 90 degrees
- renumbered J5 to J4, J6 to J5, J7 to J6, J12 to J7, J11 to J8, TP2 to TP10, TP3 to TP11, TP1 to TP9, U5 to U10, U6 to U12, U2 to U4, U1 to U5, U4 to U9
Connections:
- FPC1 pad 1: unconnected-(FPC1-Pad1) -> +24V
- FPC1 pad 10: unconnected-(FPC1-Pad10) -> /SPI_CLK
- FPC1 pad 11: unconnected-(FPC1-Pad11) -> /TFT_CS
- FPC1 pad 12: unconnected-(FPC1-Pad12) -> Net-(FPC1-Pad12)
- FPC1 pad 13: unconnected-(FPC1-Pad13) -> /DE
- FPC1 pad 14: unconnected-(FPC1-Pad14) -> /VSYNC
- FPC1 pad 15: unconnected-(FPC1-Pad15) -> /HSYNC
- FPC1 pad 16: unconnected-(FPC1-Pad16) -> /B0
- FPC1 pad 17: unconnected-(FPC1-Pad17) -> /B1
- FPC1 pad 18: unconnected-(FPC1-Pad18) -> /B2
- FPC1 pad 19: unconnected-(FPC1-Pad19) -> /B3
- FPC1 pad 2: unconnected-(FPC1-Pad2) -> /Display TFT RGB TTL/LEDK
- FPC1 pad 20: unconnected-(FPC1-Pad20) -> /B4
- FPC1 pad 21: unconnected-(FPC1-Pad21) -> /B5
- FPC1 pad 22: unconnected-(FPC1-Pad22) -> /G0
- FPC1 pad 23: unconnected-(FPC1-Pad23) -> /G1
- FPC1 pad 24: unconnected-(FPC1-Pad24) -> /G2
- FPC1 pad 25: unconnected-(FPC1-Pad25) -> /G3
- FPC1 pad 26: unconnected-(FPC1-Pad26) -> /G4
- FPC1 pad 27: unconnected-(FPC1-Pad27) -> /G5
- FPC1 pad 28: unconnected-(FPC1-Pad28) -> /R0
- FPC1 pad 29: unconnected-(FPC1-Pad29) -> /R1
- FPC1 pad 3: unconnected-(FPC1-Pad3) -> /Display TFT RGB TTL/LEDK
- FPC1 pad 30: unconnected-(FPC1-Pad30) -> /R2
- FPC1 pad 31: unconnected-(FPC1-Pad31) -> /R3
- FPC1 pad 32: unconnected-(FPC1-Pad32) -> /R4
- FPC1 pad 33: unconnected-(FPC1-Pad33) -> /R5
- FPC1 pad 34: unconnected-(FPC1-Pad34) -> GND
- FPC1 pad 35: unconnected-(FPC1-Pad35) -> /TP_IRQ
- FPC1 pad 36: unconnected-(FPC1-Pad36) -> /I2C_SCL
- FPC1 pad 37: unconnected-(FPC1-Pad37) -> /I2C_SDA
- FPC1 pad 38: unconnected-(FPC1-Pad38) -> /RST
- FPC1 pad 39: unconnected-(FPC1-Pad39) -> +3.3V
- FPC1 pad 4: unconnected-(FPC1-Pad4) -> GND
- FPC1 pad 40: unconnected-(FPC1-Pad40) -> GND
- FPC1 pad 41: unconnected-(FPC1-Pad41) -> GND
- FPC1 pad 42: unconnected-(FPC1-Pad42) -> GND
- FPC1 pad 5: unconnected-(FPC1-Pad5) -> +3.3V
- FPC1 pad 6: unconnected-(FPC1-Pad6) -> /RST
- FPC1 pad 7: unconnected-(FPC1-Pad7) -> /Display TFT RGB TTL/IM1
- FPC1 pad 8: unconnected-(FPC1-Pad8) -> /Display TFT RGB TTL/IM0
- FPC1 pad 9: unconnected-(FPC1-Pad9) -> /SPI_MOSI
- J3 pad 1: VBUS -> /TRX_P
- J3 pad 2: /USB_DBG_D_P -> /TRX_N
- J8 pad 7: /GPIO_06 -> GND
- J8 pad 8: /GPIO_07 -> /ADC1
- J8 pad 9: /GPIO_08 -> /ADC2
- J9 pad 1: +3.3V -> unconnected-(J9-Pad1)
- J9 pad 2: /ADC2 -> unconnected-(J9-Pad2)
- J9 pad 3: GND -> unconnected-(J9-Pad3)
- U10 pad 1: unconnected-(U5-GND-Pad1) -> GND
- U10 pad 13: unconnected-(U5-C6_IO5-Pad13) -> /GPIO_03
- U10 pad 14: unconnected-(U5-C6_IO4-Pad14) -> /GPIO_02
- U10 pad 15: unconnected-(U5-GND-Pad15) -> GND
- U10 pad 16: unconnected-(U5-GPIO1-Pad16) -> /SPE_CS
- U10 pad 17: unconnected-(U5-GPIO2-Pad17) -> /LAN_RESET_N
- U10 pad 18: unconnected-(U5-GPIO3-Pad18) -> /IRQ_N
- U10 pad 19: unconnected-(U5-GPIO4-Pad19) -> /GPIO_01
- U10 pad 20: unconnected-(U5-GPIO5-Pad20) -> /UART2_RX
- U10 pad 21: unconnected-(U5-GPIO6-Pad21) -> /UART2_TX
- U10 pad 22: unconnected-(U5-GPIO7-Pad22) -> /I2C_SDA
- U10 pad 23: unconnected-(U5-GPIO8-Pad23) -> /I2C_SCL
- U10 pad 24: unconnected-(U5-GPIO9-Pad24) -> /UART1_TX
- U10 pad 25: unconnected-(U5-GPIO10-Pad25) -> /UART1_RX
- U10 pad 26: unconnected-(U5-GPIO11-Pad26) -> /ESP32-P4 + C6/I2S_ASDOUT
- U10 pad 27: unconnected-(U5-GPIO12-Pad27) -> /ESP32-P4 + C6/I2S_SCLK
- U10 pad 28: unconnected-(U5-GPIO13-Pad28) -> /ESP32-P4 + C6/I2S_MCLK
- U10 pad 29: unconnected-(U5-GPIO20-Pad29) -> /CAN_INT
- U10 pad 3: unconnected-(U5-GND-Pad3) -> GND
- U10 pad 30: unconnected-(U5-GPIO21-Pad30) -> /ESP32-P4 + C6/ADC1_CHANEL5
- U10 pad 31: unconnected-(U5-GPIO22-Pad31) -> /ESP32-P4 + C6/I2S_LRCK
- U10 pad 32: unconnected-(U5-GPIO23-Pad32) -> /ESP32-P4 + C6/I2S_DSDIN
- U10 pad 33: unconnected-(U5-GND-Pad33) -> GND
- U10 pad 4: unconnected-(U5-C6_U0RXD-Pad4) -> /ESP32-P4 + C6/C6_U0RXD
- U10 pad 40: unconnected-(U5-GND-Pad40) -> GND
- U10 pad 47: unconnected-(U5-GND-Pad47) -> GND
- U10 pad 48: unconnected-(U5-USB_DM-Pad48) -> /USB_USER_D_N
- U10 pad 49: unconnected-(U5-USB_DP-Pad49) -> /USB_USER_D_P
- U10 pad 5: unconnected-(U5-C6_U0TXD-Pad5) -> /ESP32-P4 + C6/C6_U0TXD
- U10 pad 50: unconnected-(U5-GPIO24-Pad50) -> Net-(U10-GPIO24)
- U10 pad 51: unconnected-(U5-GPIO25-Pad51) -> Net-(U10-GPIO25)
- U10 pad 52: unconnected-(U5-GND-Pad52) -> GND
- U10 pad 53: unconnected-(U5-GPIO26-Pad53) -> /Backlight
- U10 pad 54: unconnected-(U5-GPIO27-Pad54) -> /R5
- U10 pad 55: unconnected-(U5-GPIO28-Pad55) -> /RST
- U10 pad 56: unconnected-(U5-GPIO29-Pad56) -> /SPI_MISO
- U10 pad 57: unconnected-(U5-GPIO30-Pad57) -> /SPI_CLK
- U10 pad 58: unconnected-(U5-GPIO31-Pad58) -> /SPI_MOSI
- U10 pad 59: unconnected-(U5-GPIO32-Pad59) -> /R4
- U10 pad 6: unconnected-(U5-C6_IO15-Pad6) -> /ESP32-P4 + C6/C6_IO15
- U10 pad 60: unconnected-(U5-GPIO33-Pad60) -> /R3
- U10 pad 61: unconnected-(U5-GPIO34-Pad61) -> /R2
- U10 pad 62: unconnected-(U5-GPIO35-Pad62) -> /BUTTON1
- U10 pad 63: unconnected-(U5-GPIO36-Pad63) -> /R1
- U10 pad 64: unconnected-(U5-GPIO37-Pad64) -> /R0
- U10 pad 65: unconnected-(U5-GPIO38-Pad65) -> /G5
- U10 pad 67: unconnected-(U5-GPIO39-Pad67) -> /G4
- U10 pad 68: unconnected-(U5-GPIO40-Pad68) -> /G3
- U10 pad 69: unconnected-(U5-GPIO41-Pad69) -> /G2
- U10 pad 7: unconnected-(U5-C6_IO14-Pad7) -> /GPIO_06
- U10 pad 70: unconnected-(U5-GPIO42-Pad70) -> /G1
- U10 pad 71: unconnected-(U5-GPIO43-Pad71) -> /G0
- U10 pad 72: unconnected-(U5-GPIO44-Pad72) -> /B5
- U10 pad 73: unconnected-(U5-GPIO45-Pad73) -> /B4
- U10 pad 74: unconnected-(U5-GPIO46-Pad74) -> /B3
- U10 pad 75: unconnected-(U5-GPIO47-Pad75) -> /B2
- U10 pad 76: unconnected-(U5-GPIO48-Pad76) -> /B1
- U10 pad 77: unconnected-(U5-GPIO49-Pad77) -> /B0
- U10 pad 78: unconnected-(U5-GPIO50-Pad78) -> /VSYNC
- U10 pad 79: unconnected-(U5-GPIO51-Pad79) -> /DE
- U10 pad 8: unconnected-(U5-C6_IO13-Pad8) -> /GPIO_05
- U10 pad 80: unconnected-(U5-GPIO52-Pad80) -> /TP_IRQ
- U10 pad 81: unconnected-(U5-GPIO53-Pad81) -> /HSYNC
- U10 pad 82: unconnected-(U5-GPIO54-Pad82) -> /PCLK
- U10 pad 83: unconnected-(U5-GND-Pad83) -> GND
- U10 pad 84: unconnected-(U5-VBAT-Pad84) -> Net-(D1-K)
- U10 pad 85: unconnected-(U5-ESP_3V3-Pad85) -> +3.3V
- U10 pad 86: unconnected-(U5-ESP_3V3-Pad86) -> +3.3V
- U10 pad 87: unconnected-(U5-ESP_EN-Pad87) -> /BUTTON2
- U10 pad 88: unconnected-(U5-GPIO0-Pad88) -> /CAN_CS
- U10 pad 9: unconnected-(U5-C6_IO9-Pad9) -> /ESP32-P4 + C6/C6_IO9
- U12 pad 1: unconnected-(U6-SW-Pad1) -> Net-(D2-A)
- U12 pad 2: unconnected-(U6-GND-Pad2) -> GND
- U12 pad 3: unconnected-(U6-FB-Pad3) -> /Display TFT RGB TTL/LEDK
- U12 pad 4: unconnected-(U6-CTRL-Pad4) -> /Backlight
- U12 pad 5: unconnected-(U6-VIN-Pad5) -> +5V
- U3 pad 1: unconnected-(U3-MCLK-Pad1) -> Net-(C1-Pad1)
- U3 pad 2: unconnected-(U3-DVDD-Pad2) -> GND
- U4 pad 1: unconnected-(U2-TXCAN-Pad1) -> Net-(U4-TXCAN)
- U4 pad 10: unconnected-(U2-SCK-Pad10) -> /SPI_CLK
- U4 pad 11: unconnected-(U2-SDI-Pad11) -> /SPI_MOSI
- U4 pad 12: unconnected-(U2-SDO-Pad12) -> /SPI_MISO
- U4 pad 13: unconnected-(U2-nCS-Pad13) -> /CAN_CS
- U4 pad 14: unconnected-(U2-VDD-Pad14) -> +3.3V
- U4 pad 2: unconnected-(U2-RXCAN-Pad2) -> Net-(U4-RXCAN)
- U4 pad 4: unconnected-(U2-~{INT}-Pad4) -> /CAN_INT
- U4 pad 7: unconnected-(U2-VSS-Pad7) -> GND
- U4 pad 8: unconnected-(U2-~{INT1}/GPIO1-Pad8) -> /CAN_INT1
- U4 pad 9: unconnected-(U2-~{INT0}/GPIO0/XSTBY-Pad9) -> /CAN_INT0
- U5 pad 1: unconnected-(U1-TXD-Pad1) -> Net-(U4-TXCAN)
- U5 pad 2: unconnected-(U1-GND-Pad2) -> GND
- U5 pad 3: unconnected-(U1-VCC-Pad3) -> +5V
- U5 pad 4: unconnected-(U1-RXD-Pad4) -> Net-(U4-RXCAN)
- U5 pad 5: unconnected-(U1-VIO-Pad5) -> +3.3V
- U5 pad 6: unconnected-(U1-CANL-Pad6) -> /CAN_L
- U5 pad 7: unconnected-(U1-CANH-Pad7) -> /CAN_H
- U5 pad 8: unconnected-(U1-STBY-Pad8) -> GND
- U9 pad 100: unconnected-(U4-VO_LCDC_D6/VI_CIF_D3_M1/PWM4_M2/SPI0_CLK_M0/SDIO_D0_M1/GPIO1_C1_d-Pad100) -> /G0
- U9 pad 101: unconnected-(U4-VO_LCDC_D7/VI_CIF_D2_M1/PWM2_M2/SPI0_CS0_M0/SDIO_D1_M1/GPIO1_C0_d-Pad101) -> /G1
- U9 pad 102: unconnected-(U4-SDIO_D1_M0/I2S0_SCLK/VO_LCDC_D8/UART1_CTS_M1/I2C4_SDA_M0/GPIO2_A0_d-Pad102) -> /G2
- U9 pad 103: unconnected-(U4-SDIO_D0_M0/I2S0_LRCK/VO_LCDC_D9/UART1_RTS_M1/I2C4_SCL_M0/GPIO2_A1_d-Pad103) -> /G3
- U9 pad 104: unconnected-(U4-SDIO_CLK_M0/I2S0_MCLK/VO_LCDC_D10/GPIO2_A2_d-Pad104) -> /G4
- U9 pad 105: unconnected-(U4-SDIO_CMD_M0/I2S0_SDO3_SDI1/VO_LCDC_D11/GPIO2_A3_d-Pad105) -> /G5
- U9 pad 106: unconnected-(U4-SDIO_D3_M0/I2S0_SDO0/VO_LCDC_D12/UART1_TX_M1/GPIO2_A4_d-Pad106) -> /R0
- U9 pad 107: unconnected-(U4-SDIO_D2_M0/I2S0_SDI0/VO_LCDC_D13/UART1_RX_M1/GPIO2_A5_d-Pad107) -> /R1
- U9 pad 108: unconnected-(U4-UART0_RTS_M1/I2S0_SDO2_SDI2/VO_LCDC_D14/PWM2_M1/I2C3_SCL_M0/FLASH_TRIG_OUT/GPIO2_A6_d-Pad108) -> /R2
- U9 pad 109: unconnected-(U4-UART0_CTS_M1/I2S0_SDO1_SDI3/VO_LCDC_D15/PWM4_M1/I2C3_SDA_M0/PRELIGHT_TRIG_OUT/GPIO2_A7_d-Pad109) -> /R3
- U9 pad 110: unconnected-(U4-UART0_RX_M1/I2C1_SCL_M1/VO_LCDC_D16/PWM5_M1/GPIO2_B0_d-Pad110) -> /R4
- U9 pad 111: unconnected-(U4-UART0_TX_M1/I2C1_SDA_M1/VO_LCDC_D17/PWM6_M1/GPIO2_B1_d-Pad111) -> /R5
- U9 pad 112: unconnected-(U4-GND-Pad112) -> GND
- U9 pad 21: unconnected-(U4-GND-Pad21) -> GND
- U9 pad 22: unconnected-(U4-USB_N-Pad22) -> /USB_USER_D_N
- U9 pad 23: unconnected-(U4-USB_P-Pad23) -> /USB_USER_D_P
- U9 pad 25: unconnected-(U4-GND-Pad25) -> GND
- U9 pad 26: unconnected-(U4-SARADC_IN0/GPIO4_C0_z-Pad26) -> /BUTTON1
- U9 pad 27: unconnected-(U4-SARADC_IN1/PWM1_M1/GPIO4_C1_z-Pad27) -> /Core1106/ADC1
- U9 pad 28: unconnected-(U4-GND-Pad28) -> GND
- U9 pad 29: unconnected-(U4-GND-Pad29) -> GND
- U9 pad 36: unconnected-(U4-GND-Pad36) -> GND
- U9 pad 41: unconnected-(U4-EMMC_D4/SPI1_CS0_M0/UART1_TX_M2/I2C2_SDA_M1/GPIO4_A5_u-Pad41) -> /CAN_CS
- U9 pad 42: unconnected-(U4-EMMC_D5/SPI1_CLK_M0/UART1_RX_M2/I2C2_SCL_M1/GPIO4_A7_u-Pad42) -> /SPI_CLK
- U9 pad 43: unconnected-(U4-EMMC_D6/SPI1_MOSI_M0/UART0_TX_M2/I2C0_SCL_M1/GPIO4_A1_u-Pad43) -> /SPI_MOSI
- U9 pad 44: unconnected-(U4-EMMC_D7/SPI1_MISO_M0/UART0_RX_M2/I2C0_SDA_M1/GPIO4_A0_u-Pad44) -> /SPI_MISO
- U9 pad 47: unconnected-(U4-GND-Pad47) -> GND
- U9 pad 48: unconnected-(U4-SDMMC_DET/GPIO3_A1_u-Pad48) -> /TFT_CS
- U9 pad 49: unconnected-(U4-SDMMC_D0/UART2_RX_M0/PWM8_M0/GPIO3_A3_u-Pad49) -> /GPIO_01
- U9 pad 50: unconnected-(U4-SDMMC_D1/UART2_TX_M0/PWM9_M0/GPIO3_A2_u-Pad50) -> /GPIO_02
- U9 pad 51: unconnected-(U4-SDMMC_D2/UART5_RX_M0/JTAG_CPU_TCK_M0/JTAG_HPMCU_TCK_M1/GPIO3_A7_u-Pad51) -> /GPIO_05
- U9 pad 52: unconnected-(U4-SDMMC_D3/UART5_TX_M0/JTAG_CPU_TMS_M0/JTAG_HPMCU_TMS_M1/GPIO3_A6_u-Pad52) -> /GPIO_06
- U9 pad 53: unconnected-(U4-SDMMC_CMD/UART5_CTS_M0/I2C0_SDA_M2/JTAG_LPMCU_TMS_M1/PWM11_IR_M0/GPIO3_A5_u-Pad53) -> /GPIO_04
- U9 pad 54: unconnected-(U4-SDMMC_CLK/UART5_RTS_M0/I2C0_SCL_M2/JTAG_LPMCU_TCK_M1/PWM10_M0/GPIO3_A4_d-Pad54) -> /GPIO_03
- U9 pad 55: unconnected-(U4-GND-Pad55) -> GND
- U9 pad 56: unconnected-(U4-GND-Pad56) -> GND
- U9 pad 57: unconnected-(U4-GND-Pad57) -> GND
- U9 pad 58: unconnected-(U4-UART0_RX_M0/CLK_32K/CLK_REFOUT/RTC_CLKO/GPIO0_A0_z-Pad58) -> Net-(U9-UART0_RX_M0/CLK_32K/CLK_REFOUT/RTC_CLKO/GPIO0_A0_z)
- U9 pad 59: unconnected-(U4-UART0_TX_M0/PWM2_M0/GPIO0_A1_d-Pad59) -> Net-(U9-UART0_TX_M0/PWM2_M0/GPIO0_A1_d)
- U9 pad 61: unconnected-(U4-PWR_CTRL_M1/GPIO0_A3_u-Pad61) -> /Core1106/GPIO0_A3
- U9 pad 62: unconnected-(U4-PWR_CTRL_M0/PWM1_M0/GPIO0_A4_d-Pad62) -> /SPE_CS
- U9 pad 63: unconnected-(U4-I2C1_SCL_M0/UART1_RTS_M0/PWM5_M0/GPIO0_A5_d-Pad63) -> /I2C_SCL
- U9 pad 64: unconnected-(U4-I2C1_SDA_M0/UART1_CTS_M0/PWM6_M0/GPIO0_A6_d-Pad64) -> /I2C_SDA
- U9 pad 65: unconnected-(U4-UART3_TX_M0/I2C2_SCL_M0/PWM7_IR_M0/GPIO1_A0_d-Pad65) -> /UART2_RX
- U9 pad 66: unconnected-(U4-UART3_RX_M0/I2C2_SDA_M0/PMU_DEBUG/PWM4_M0/GPIO1_A1_d-Pad66) -> /UART2_TX
- U9 pad 67: unconnected-(U4-PWM0_M0/CPU_AVS/VI_CIF_D0_M1/GPIO1_A2_d-Pad67) -> /TP_IRQ
- U9 pad 68: unconnected-(U4-UART1_TX_M0/I2C0_SCL_M0/GPIO1_A3_d-Pad68) -> /UART1_TX
- U9 pad 69: unconnected-(U4-UART1_RX_M0/I2C0_SDA_M0/GPIO1_A4_d-Pad69) -> /UART1_RX
- U9 pad 70: unconnected-(U4-UART4_RX_M0/PWM3_IR_M1/GPIO1_B0_d-Pad70) -> /Backlight
- U9 pad 71: unconnected-(U4-UART4_TX_M0/PWM7_IR_M1/SPI1_CS1_M0/VI_CIF_D1_M1/GPIO1_B1_d-Pad71) -> /RST
- U9 pad 72: unconnected-(U4-JTAG_CPU_TCK_M1/UART2_TX_M1/JTAG_HPMCU_TCK_M0/JTAG_LPMCU_TCK_M0/GPIO1_B2_d-Pad72) -> Net-(U9-JTAG_CPU_TCK_M1/UART2_TX_M1/JTAG_HPMCU_TCK_M0/JTAG_LPMCU_TCK_M0/GPIO1_B2_d)
- U9 pad 73: unconnected-(U4-JTAG_CPU_TMS_M1/UART2_RX_M1/JTAG_HPMCU_TMS_M0/JTAG_LPMCU_TMS_M0/GPIO1_B3_u-Pad73) -> Net-(U9-JTAG_CPU_TMS_M1/UART2_RX_M1/JTAG_HPMCU_TMS_M0/JTAG_LPMCU_TMS_M0/GPIO1_B3_u)
- U9 pad 74: unconnected-(U4-NPOR-Pad74) -> /BUTTON2
- U9 pad 75: unconnected-(U4-GND-Pad75) -> GND
- U9 pad 76: unconnected-(U4-VCC3V3_RTC-Pad76) -> +3.3V
- U9 pad 77: unconnected-(U4-VCC_1V8-Pad77) -> +1V8
- U9 pad 78: unconnected-(U4-VCC_3V3-Pad78) -> +3.3V
- U9 pad 79: unconnected-(U4-VCC5V0_SYS-Pad79) -> +5V
- U9 pad 80: unconnected-(U4-VCC5V0_SYS-Pad80) -> +5V
- U9 pad 81: unconnected-(U4-VCC5V0_SYS-Pad81) -> +5V
- U9 pad 82: unconnected-(U4-GND-Pad82) -> GND
- U9 pad 83: unconnected-(U4-GND-Pad83) -> GND
- U9 pad 84: unconnected-(U4-GND-Pad84) -> GND
- U9 pad 89: unconnected-(U4-GND-Pad89) -> GND
- U9 pad 90: unconnected-(U4-VO_LCDC_CLK/VI_CIF_CLKO_M1/I2C3_SCL_M1/UART5_TX_M1/PWM11_IR_M2/AUD_DSM_N/GPIO1_D3_d-Pad90) -> /PCLK
- U9 pad 91: unconnected-(U4-VO_LCDC_VSYNC/VI_CIF_VSYNC_M1/I2C3_SDA_M1/UART5_RX_M1/SPI0_CS1_M0/PWM0_M1/AUD_DSM_P/GPIO1_D2_d-Pad91) -> /VSYNC
- U9 pad 92: unconnected-(U4-VO_LCDC_HSYNC/VI_CIF_HREF_M1/PWM10_M2/UART5_CTS_M1/UART3_RX_M1/GPIO1_D1_d-Pad92) -> /HSYNC
- U9 pad 93: unconnected-(U4-VO_LCDC_DEN/VI_CIF_CLKI_M1/PWM3_IR_M2/UART5_RTS_M1/UART3_TX_M1/GPIO1_D0_d-Pad93) -> /DE
- U9 pad 94: unconnected-(U4-VO_LCDC_D0/VI_CIF_D9_M1/PWM11_IR_M1/UART4_CTS_M1/GPIO1_C7_d-Pad94) -> /B0
- U9 pad 95: unconnected-(U4-VO_LCDC_D1/VI_CIF_D8_M1/PWM10_M1/UART4_RTS_M1/GPIO1_C6_d-Pad95) -> /B1
- U9 pad 96: unconnected-(U4-VO_LCDC_D2/VI_CIF_D7_M1/PWM9_M1/UART4_TX_M1/SDIO_D2_M1/GPIO1_C5_d-Pad96) -> /B2
- U9 pad 97: unconnected-(U4-VO_LCDC_D3/VI_CIF_D6_M1/PWM8_M1/UART4_RX_M1/SDIO_D3_M1/GPIO1_C4_d-Pad97) -> /B3
- U9 pad 98: unconnected-(U4-VO_LCDC_D4/VI_CIF_D5_M1/PWM6_M2/I2C4_SDA_M1/SDIO_CMD_M1/SPI0_MISO_M0/GPIO1_C3_d-Pad98) -> /B4
- U9 pad 99: unconnected-(U4-VO_LCDC_D5/VI_CIF_D4_M1/PWM5_M2/I2C4_SCL_M1/SDIO_CLK_M1/SPI0_MOSI_M0/GPIO1_C2_d-Pad99) -> /B5
Routing:
- net +3V3: track 0.00 -> 43.1 mm, vias 0 -> 5
- net GND: track 0.00 -> 39.9 mm, vias 0 -> 8
- net (no net): track 0.00 -> 30.8 mm, vias 0 -> 2
- net /SPI_CLK: track 0.00 -> 22.7 mm, vias 0 -> 1
- net /SPI_MOSI: track 0.00 -> 22.7 mm, vias 0 -> 1
- net /SPI_MISO: track 0.00 -> 20.6 mm, vias 0 -> 2
- net Net-(U1-VDDA): track 0.00 -> 11.6 mm
- net /LAN_RESET_N: track 0.00 -> 9.10 mm, vias 0 -> 1
- net /IRQ_N: track 0.00 -> 9.09 mm, vias 0 -> 1
- net /SPE_CS: track 0.00 -> 8.11 mm, vias 0 -> 2
- net /XTI: track 0.00 -> 6.51 mm
- net /TRX_P: track 0.00 -> 4.68 mm
- net Net-(C2-Pad1): track 0.00 -> 4.36 mm
- net /TRX_N: track 0.00 -> 4.31 mm
- net Net-(C1-Pad1): track 0.00 -> 4.29 mm
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Other:
- copper layers 2 -> 4
