File: Electronic/DisplayTTL/DisplayTTL.kicad_sch (KiCad schematic)
At the start: 19 parts, among them J1 Conn_01x05, J10 Conn_01x03, J11 Conn_01x10, J12 Conn_01x02, J2 Conn_01x04, J3 Conn_01x04, J4 TC2050, J5 Conn_01x02, J6 Conn_01x04, J7 Conn_01x04, J8 Conn_01x02, J9 Conn_01x03, U1 ATA6563-GAQW1, U2 MCP2518FDT-E/SL, U3 ES8388

Commit message: Add RV1106 RGB666 pinout doc: bus mapping, pin allocation, GPIO recovery plan
Schematic:
- Wire most of the gpios,
- Button for boot / reset
- DIsplay schematic done
- Wip I2S codec wiring on ESP32-P4 side
- Single Pair Ethernet T1S
- I2C ADC with 4 input
- Core1106 / ESP32-P4 wiring mostly done

WIP PCB layout / schematic.

Docs:
- Add Pico Pi schematic (use the Core1106 module)
- Add Makerworld url for stick and stick position
Parts:
- removed J10, J9: Conn_01x03, Connector_PinSocket_2.54mm:PinSocket_1x03_P2.54mm_Vertical, symbol Connector:Conn_01x03_Socket
- removed J3: Conn_01x04, Connector_PinSocket_2.54mm:PinSocket_1x04_P2.54mm_Vertical, symbol Connector:Conn_01x04_Socket
- removed J4: TC2050, Connector:Tag-Connect_TC2050-IDC-NL_2x05_P1.27mm_Vertical, symbol Connector:TC2050
- removed J8: Conn_01x02, Connector_PinSocket_2.54mm:PinSocket_1x02_P2.54mm_Vertical, symbol Connector:Conn_01x02_Socket
- removed U3: ES8388, Package_DFN_QFN:QFN-28-1EP_4x4mm_P0.45mm_EP2.6x2.6mm, symbol Audio:ES8388
- added C1, C10, C11, C2, C3, C5, C7, C8: 0.1uF, Capacitor_SMD:C_0201_0603Metric, symbol Device:C
- added C12, C18, C23, C24, C4: 0.1uF, Capacitor_SMD:C_0402_1005Metric, symbol Device:C
- added C13, C9: 10pF, Capacitor_SMD:C_0201_0603Metric, symbol Device:C
- added C14, C15, C16, C17: 10nF, Capacitor_SMD:C_0201_0603Metric, symbol Device:C
- added C19, C20, C21, C22: 10uF, Capacitor_SMD:C_0402_1005Metric, symbol Device:C
- added C6: 4.7uF, Capacitor_SMD:C_0402_1005Metric, symbol Device:C
- added J3: Conn_01x02, Connector_PinSocket_2.54mm:PinSocket_1x02_P2.54mm_Vertical, symbol Connector:Conn_01x02_Socket
- added JP1, JP2: Jumper_2_Open, Jumper:SolderJumper-2_P1.3mm_Open_RoundedPad1.0x1.5mm, symbol Jumper:Jumper_2_Open
- added JP3: Jumper_3_Open, symbol Jumper:Jumper_3_Open
- added L1: DLW32MH201XK2L, lcsc:FILTER-SMD_4P-L3.2-W2.5-BL_DLW32SH510XK2L, symbol lcsc:DLW32MH201XK2L
- added L2: BLM18KG331SN1D, lcsc:L0603, symbol lcsc:BLM18KG331SN1D
- added R1, R4: 100K, Resistor_SMD:R_0201_0603Metric, symbol Device:R
- added R10, R11, R8, R9: 10K, symbol Device:R
- added R2, R3: 49.9R, Resistor_SMD:R_0201_0603Metric, symbol Device:R
- added R5: 12.4K 1%, Resistor_SMD:R_0201_0603Metric, symbol Device:R
- added R6: 10K, Resistor_SMD:R_0201_0603Metric, symbol Device:R
- added R7: 120R, symbol Device:R
- added SW1, SW2: SH-1808SN-250GF, lcsc:SW-SMD_4P-L4.2-W3.4-P2.15-LS5.2, symbol lcsc:SH-1808SN-250GF
- added TP1, TP2, TP3, TP4: TestPoint, TestPoint:TestPoint_Pad_D1.5mm, symbol Connector:TestPoint
- added U1: LAN8651B1-E/LMX, lcsc:VQFN-32_L5.0-W5.0-P0.50-TL-EP3.6, symbol lcsc:LAN8651B1-E_LMX
- added U2, U3: AVRH10C221KT1R5YA8, lcsc:R0402, symbol lcsc:AVRH10C221KT1R5YA8
- added U6, U7: ESD5451N_C5261080, lcsc:DFN1006-2L-BI, symbol lcsc:ESD5451N_C5261080
- added U8: ADS1115IDGSR, lcsc:MSOP-10_L3.0-W3.0-P0.50-LS5.0-BL, symbol lcsc:ADS1115IDGSR
- added X1: ABM10-25.000MHZ-D30-T3, lcsc:CRYSTAL-SMD_4P-L2.5-W2.0-BL-B, symbol lcsc:ABM10-25.000MHZ-D30-T3
- renumbered J5 to J4, J6 to J5, J7 to J6, J12 to J7, J11 to J8, U2 to U4, U1 to U5
Connections:
- net GPIO_07 is gone; now on net ADC1: J8.8 (Pin_8)
- net GPIO_08 is gone; now on net ADC2: J8.9 (Pin_9)
- net +3.3V: now also U4.14 (VDD), U5.5 (VIO), C12.1, C18.1, C23.1, R11.1, R8.1, R9.1, U8.8 (VDD)
- net +5V: now also U5.3 (VCC), C4.1
- net ADC1: now also U8.5 (AIN1)
- net CAN_H: now also U5.7 (CANH), R7.1
- net CAN_L: now also U5.6 (CANL), R7.2
- net GND: now also J8.7 (Pin_7), U4.7 (VSS), U5.2 (GND), U5.8 (STBY), C10.2, C11.2, C12.2, C13.2, C14.2, C15.2, C16.2, C17.2, C18.2, C19.2, C20.2, C21.2, C22.2, C23.2, C24.2, C4.2, C6.2, C7.2, C8.2, C9.2, JP1.1 (A), JP2.1 (A), R5.2, SW1.3, SW1.4, SW2.3, SW2.4, U1.14 (DIOB1), U1.2 (VSS), U1.3 (VSS), U1.32 (WAKE_IN), U1.33 (EP), U1.5 (VSS), U2.1, U3.2, U6.1, U7.1, U8.1 (ADDR), U8.3 (GND), X1.2 (GND), X1.4 (GND)
- net GPIO_06: no longer J8.7 (Pin_7)
- net SPI_CLK: now also U4.10 (SCK), U1.12 (SCLK)
- net SPI_MISO: now also U4.12 (SDO), U1.10 (SDO)
- net SPI_MOSI: now also U4.11 (SDI), U1.13 (SDI)
- net at U5.1 (TXD): now also U4.1 (TXCAN)
- net at U5.4 (RXD): now also U4.2 (RXCAN)
- net CAN_CS: now reaches U4.13 (nCS)
- net CAN_INT: now reaches U4.4 (~{INT})
- net CAN_INT1: now reaches U4.8 (~{INT1}/GPIO1)
- net CAN_INT0: now reaches U4.9 (~{INT0}/GPIO0/XSTBY)
- new net: C1.2, L1.2
- new net: C2.2, L1.3
- new net: C2.1, R2.1, TP4.1, U2.2
- new net: C1.1, R3.1, TP3.1, U3.1
- new net: JP3.1 (A), R10.2
- new net: C3.1, R1.1, R2.2
- new net: C3.2, JP1.2 (B), R1.2
- new net: C10.1, C14.1, C16.1, C19.1, C21.1, C7.1, L2.2, U1.25 (VDDAU), U1.29 (VDDA)
- new net: C5.1, R3.2, R4.1
- new net: JP3.3 (B), R11.2
- new net: C6.1, U1.21 (CCOMP)
- new net: R5.1, U1.26 (RBIAS)
- new net: C5.2, JP2.2 (B), R4.2
- new net +1V8: R10.1
- new net +3V3: C11.1, C15.1, C17.1, C20.1, C22.1, C8.1, L2.1, R6.2, U1.17 (VDDP), U1.4 (TEST), U1.7 (VDDP)
- new net ADC0: U8.4 (AIN0)
- new net ADC3: U8.7 (AIN3)
- new net ADC4: U8.6 (AIN2)
- new net BUTTON1: SW1.1, SW1.2, U6.2
- new net BUTTON2: C24.1, JP3.2 (C), SW2.1, SW2.2, U7.2
- new net DIOA0: TP2.1, U1.18 (DIOA0)
- new net DIOA1: TP1.1, U1.19 (DIOA1)
- new net DIOA2: U1.20 (DIOA2)
- new net DIOA3: U1.22 (DIOA3)
- new net DIOA4: U1.23 (DIOA4)
- new net DIOB0: U1.16 (DIOB0)
- new net I2C_SCL: R8.2, U8.10 (SCL)
- new net I2C_SDA: R9.2, U8.9 (SDA)
- new net IRQ_N: R6.1, U1.9 (RQ_N)
- new net LAN_RESET_N: U1.8 (RESET_N)
- new net SPE_CS: U1.11 (CS_N)
- new net TRX_N: J3.2 (Pin_2), L1.4, U1.31 (TRXN)
- new net TRX_P: J3.1 (Pin_1), L1.1, U1.30 (TRXP)
- new net XTI: C13.1, U1.27 (XTI), X1.3 (OSC2)
- new net XTO: C9.1, U1.28 (XTO), X1.1 (OSC1)
- no-connect marks 0 -> 5
Other:
- sheet Core1106 ports: added ADC0, ADC1, BOOT, GPIO0_A3, GPIO0_A4, GPIO3_A1, GPIO3_A2, GPIO3_A4, GPIO3_A5, GPIO3_A6, GPIO3_A7, GPIO4_A5, I2C1_SCL, I2C1_SDA, RESET, SPI1_CLK, SPI1_MISO, SPI1_MOSI, TFT_CS, UART1_RX, UART1_TX, UART3_RX, UART3_TX, USB_D_N, USB_D_P; removed I2C0_SCL, I2C0_SDA
- sheet Display TFT RGB TTL ports: added BACKLIGHT_PWM; removed none
- sheet ESP32-P4 + C6 ports: added ADC1_CHANEL4, ADC1_CHANEL5, B0, B1, B2, B3, B4, B5, BOOT, C6_IO13, C6_IO14, C6_IO15, C6_IO4, C6_IO5, C6_IO6, DE, G0, G1, G2, G3, G4, G5, GPIO0, GPIO1, GPIO2, GPIO3, GPIO4, HSYNC, I2C_SCL, I2C_SDA, PCLK, PWM_Backlight, R0, R1, R2, R3, R4, R5, RESET, SPI_CLK, SPI_MISO, SPI_MOSI, TFT_EN, TFT_RST, UART1_RX, UART1_TX, UART2_RX, UART2_TX, USB_HS_N, USB_HS_P, VSYNC; removed none
- note added: "CAN-FD"
- note added: "Single Pair Ethernet T1S"
- note added: "TODO : - Current limiter - ESD / surge protection - Power supply"
- moved on the sheet: J4, J5, J6, J7, J8, U4, U5
