File: Electronic/Satellite/Satellite.kicad_sch (KiCad schematic)
At the start: 134 parts, among them CN1 SM04B-SRSS-TB, CN2 SM04B-SRSS-TB, J1 Conn02_Pin, J2 Conn02_Pin, J3 Conn02_Pin, J4 Conn02_Pin, J5 TC2050, J6 Conn_01x12_Pin, J7 Conn_01x12_Pin, SW1 TS-1088-AR02016, SW2 TS-1088-AR02016, U1 LAN8651B1-E/LMX, U10 SRR1280-560M, U11 NCP1117ST33T3G, U12 RP2354A, U13 WS2812C-2020-V6, U2 AVRH10C221KT1R5YA8, U3 MCP2518FDT-E/SL, U4 ATA6563-GAQW1, U5 AVRH10C221KT1R5YA8, U6 SY8513FCC, U7 MAX3232IPWR, U8 AL8860QMP-13, U9 ABM8-272-T3_C20625731, X1 ABM10-25.000MHZ-D30-T3

Commit message: WIP Satellite : reduce cob led current, layout + routing progress
Parts:
- removed L2: NR6045T100M, lcsc:IND-SMD_L6.0-W6.0_NR6045, symbol lcsc:NR6045T100M
- removed TP3, TP4: TestPoint, TestPoint:TestPoint_Pad_D1.5mm, symbol Connector:TestPoint
- removed U10: SRR1280-560M, lcsc:IND-SMD_L12.5-W12.5-SRR1280-150M, symbol lcsc:SRR1280-560M
- removed U8: AL8860QMP-13, lcsc:MSOP-8_L3.0-W3.0-P0.65-LS4.9-BL-EP, symbol lcsc:AL8860QMP-13
- added C30, C31, C32, C33, C34: 0.1uF, Capacitor_SMD:C_0402_1005Metric, symbol Device:C
- added C43: 1uF, Capacitor_SMD:C_0402_1005Metric, symbol Device:C
- added L2: APH303020C100MP03, lcsc:IND-SMD_L3.0-W3.0_FTC303012D, symbol lcsc:APH303020C100MP03
- added L4: ABG08A40M560, lcsc:IND-SMD_L8.0-W8.0_ABG08A40, symbol lcsc:ABG08A40M560
- added U8: AL8860WT-7, lcsc:SOT-23-5_L3.0-W1.7-P0.95-LS2.8-BR, symbol lcsc:AL8860WT-7
- C10, C11, C13, C14, C15, C16, C17, C18, C20, C21, C3, C4, C5, C7: footprint Capacitor_SMD:C_0201_0603Metric -> Capacitor_SMD:C_0402_1005Metric
- R1, R2, R3, R4, R5, R6: footprint Resistor_SMD:R_0201_0603Metric -> Resistor_SMD:R_0402_1005Metric
- renumbered C33 to C35, C30 to C36, C31 to C37, C32 to C38, C34 to C39, C35 to C40, C36 to C41, C37 to C42, C38 to C44, C39 to C45, C40 to C46, C41 to C47, C42 to C48, C43 to C49, C44 to C50, C45 to C51, C46 to C52, C47 to C53, C48 to C54, L4 to L5, R15 to R14, R14 to R15, U11 to U10, U12 to U11, U13 to U12
Connections:
- net +3.3V is gone; now on net +3V3: C12.1, C19.1, U3.14 (VDD), U4.5 (VIO)
- net CLK is gone; now on net SPI1_SCK: U1.12 (SCLK)
- net MISO is gone; now on net SPI1_RX: U1.10 (SDO)
- net MOSI is gone; now on net SPI1_TX: U1.13 (SDI)
- net +3V3: now also U7.16 (VCC), C34.1
- net +5V: now also C46.1, JP3.2 (C), U10.3 (INPUT); no longer C27.1, C28.1, C29.1, JP3.3 (B), R12.1
- net 5V: no longer C46.1, JP3.2 (C), U10.3 (INPUT)
- net CAN_CS: now also U11.36 (GPIO24)
- net CAN_INT: now also U11.19 (GPIO15)
- net CAN_INT0: now also U11.34 (GPIO22)
- net CAN_INT1: now also U11.35 (GPIO23)
- net COB_SET: now also U8.4 (SET)
- net GND: now also U7.15 (GND), C32.1, C33.1, C34.2, C43.2, U8.2 (GND)
- net IRQ_N: now also U11.13 (GPIO9)
- net LAN_CS: now also U11.17 (GPIO13)
- net LAN_RESET_N: now also U11.12 (GPIO8)
- net PWM_COB: now also U8.3 (CTRL)
- net TRX_N: no longer J1.2 (Pin_2)
- net TRX_P: no longer J1.1 (Pin_1)
- net VCC: now also C43.1, U8.5 (VIN)
- net at C22.2, U6.8 (LX): now also L2.1
- net at C4.1, R2.1, U2.2: now also J1.1 (Pin_1)
- net at C3.1, R3.1, U5.1: now also J1.2 (Pin_2)
- net at U7.1 (C1+): now also C30.1
- net at U7.2 (V+): now also C33.2
- net at U7.3 (C1-): now also C30.2
- net at U7.4 (C2+): now also C31.1
- net at U7.5 (C2-): now also C31.2
- net at U7.6 (V-): now also C32.2
- net at C35.2, J4.1 (Pin_1): now also L4.2
- net at D1.2 (A): now also L4.1, U8.1 (SW)
- new net: C27.1, C28.1, C29.1, JP3.3 (B), L2.2, R12.1
- no-connect marks 16 -> 19
Other:
- moved on the sheet: C1, C10, C11, C12, C13, C14, C15, C16, C17, C18, C19, C2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

Commit message: WIP Satellite : split into multiple board for ease of debug / simplification
Parts:
- removed C12, C19, C2, C30, C31, C32, C33, C34: 0.1uF, Capacitor_SMD:C_0402_1005Metric, symbol Device:C
- removed C35, C43: 1uF, Capacitor_SMD:C_0402_1005Metric, symbol Device:C
- removed CN1, CN2: SM04B-SRSS-TB, lcsc:CONN-SMD_4P-P1.00_SM04B-SRSS-TB-LF-SN, symbol lcsc:SM04B-SRSS-TB
- removed D1: MBRS240LT3G, lcsc:SMB_L4.6-W3.6-LS5.3-RD, symbol lcsc:MBRS240LT3G
- removed J1, J2, J3, J4: Conn02_Pin, Connector_PinSocket_2.54mm:PinSocket_1x02_P2.54mm_Vertical, symbol Connector:Conn_01x02_Pin
- removed J5: TC2050, Connector:Tag-Connect_TC2050-IDC-NL_2x05_P1.27mm_Vertical, symbol Connector:TC2050
- removed J6, J7: Conn_01x12_Pin, Connector_PinSocket_2.54mm:PinSocket_1x12_P2.54mm_Vertical, symbol Connector:Conn_01x12_Pin
- removed JP3: Jumper_3_Open, Jumper:SolderJumper-3_P1.3mm_Open_RoundedPad1.0x1.5mm, symbol Jumper:Jumper_3_Open
- removed L4: ABG08A40M560, lcsc:IND-SMD_L8.0-W8.0_ABG08A40, symbol lcsc:ABG08A40M560
- removed R15: 0.066R, Resistor_SMD:R_0402_1005Metric, symbol Device:R
- removed R7: 120R, Resistor_SMD:R_0402_1005Metric, symbol Device:R
- removed TP7: TP, TestPoint:TestPoint_Pad_D1.5mm, symbol Connector:TestPoint
- removed U3: MCP2518FDT-E/SL, lcsc:SOIC-14_L8.7-W3.9-P1.27-LS6.0-BL, symbol lcsc:MCP2518FDT-E_SL
- removed U4: ATA6563-GAQW1, lcsc:SOIC-8_L4.9-W3.9-P1.27-LS6.0-BL, symbol lcsc:ATA6563-GAQW1
- removed U7: MAX3232IPWR, lcsc:TSSOP-16_L5.0-W4.4-P0.65-LS6.4-TL, symbol lcsc:MAX3232IPWR
- removed U8: AL8860WT-7, lcsc:SOT-23-5_L3.0-W1.7-P0.95-LS2.8-BR, symbol lcsc:AL8860WT-7
- added J3, J4, J5: Conn_01x10, Connector_PinSocket_2.54mm:PinSocket_1x10_P2.54mm_Vertical, symbol Connector_Generic:Conn_01x10
- added JP5, JP6, JP7, JP8: JO, Jumper:SolderJumper-2_P1.3mm_Open_RoundedPad1.0x1.5mm, symbol Jumper:Jumper_2_Open
- added TP3, TP4, TP5: TP, TestPoint:TestPoint_Pad_D1.5mm, symbol Connector:TestPoint
- renumbered C11 to C10, C13 to C11, C14 to C12, C15 to C13, C16 to C14, C17 to C15, C18 to C16, C22 to C17, C20 to C18, C21 to C19, C6 to C2, C27 to C20, C23 to C21, C24 to C22, C25 to C23, C26 to C24, C28 to C25, C29 to C26, C36 to C27, C37 to C28, C38 to C29, C40 to C30, C41 to C31, C42 to C32, C44 to C33, C45 to C34, C47 to C35, C48 to C36, C49 to C37, C50 to C38, C46 to C40, C51 to C41, C52 to C42, C53 to C43, C54 to C44, C8 to C6, C9 to C8, C10 to C9, D2 to D1, JP6 to JP10, JP7 to JP11, JP8 to JP12, JP9 to JP13, JP5 to JP9, L5 to L4, R9 to R10, R12 to R11, R13 to R12, R14 to R13, R16 to R14, R17 to R15, R18 to R16, R19 to R17, R20 to R18, R21 to R19, R10 to R2, R22 to R20, R23 to R21, R24 to R22, R25 to R23, R26 to R24, R27 to R25, R28 to R26, R29 to R27, R30 to R28, R31 to R29, R11 to R3, R32 to R30, R33 to R31, R34 to R32, R2 to R4, R3 to R5, R4 to R6, R5 to R7, R6 to R9, TP5 to TP6, TP6 to TP7, U5 to U3, U6 to U4, U9 to U5, U10 to U6, U11 to U7, U12 to U8
Connections:
- net +3V3: now also J3.3 (Pin_3)
- net +5V: now also C20.1, C25.1, C26.1, L2.2, R11.1
- net 5V: now also J3.2 (Pin_2)
- net ADC2: now also J4.10 (Pin_10)
- net ADC3: now also J3.9 (Pin_9)
- net GND: now also J3.10 (Pin_10), J5.10 (Pin_10)
- net GPIO17: now also J5.7 (Pin_7)
- net GPIO6: now also J5.1 (Pin_1)
- net GPIO7: now also J5.2 (Pin_2)
- net GPIO8: now also J5.3 (Pin_3)
- net I2C0_SCL: now also J4.2 (Pin_2), JP6.1 (A); no longer R25.1
- net I2C0_SDA: now also J4.1 (Pin_1), JP5.1 (A); no longer R24.1
- net I2C1_SCL: now also J4.4 (Pin_4), JP8.1 (A); no longer R27.1
- net I2C1_SDA: now also J4.3 (Pin_3), JP7.1 (A); no longer R26.1
- net LED_Data_Out: now also J4.5 (Pin_5)
- net RS232_TX: now also J5.4 (Pin_4), J5.5 (Pin_5)
- net RUN: now also TP5.1
- net SPI0_RX: now also J5.6 (Pin_6)
- net SPI0_SCK: now also J5.8 (Pin_8)
- net SPI0_TX: now also J5.9 (Pin_9)
- net SWCLK: now also TP4.1
- net SWDIO: now also TP3.1
- net UART1_RX: now also J4.7 (Pin_7)
- net UART1_TX: now also J4.6 (Pin_6)
- net SPE_N: now reaches C4.1, R4.1, U2.2
- net SPE_P: now reaches C3.1, R5.1, U3.1
- net at JP4.2 (C): now also J4.8 (Pin_8)
- net +12V: now reaches C1.1, C2.1, C6.1, R10.2, U4.1 (IN)
- net +12V: now also J3.1 (Pin_1)
- net at R19.2: now also J4.9 (Pin_9)
- new net: JP6.2 (B), R25.1
- new net: JP5.2 (B), R24.1
- new net: JP8.2 (B), R27.1
- new net: JP7.2 (B), R26.1
- no-connect marks 19 -> 11
Other:
- note removed: "CAN-FD"
- moved on the sheet: R2, R3, USB1

Commit message: Satellite PCB done !!!!!! (need verification)
Parts:
- removed JP4: Jumper_3_Open, Jumper:SolderJumper-3_P1.3mm_Open_RoundedPad1.0x1.5mm, symbol Jumper:Jumper_3_Open
- removed R22: 4.7K, Resistor_SMD:R_0402_1005Metric, symbol Device:R
- removed TP7: TP, TestPoint:TestPoint_Pad_D1.5mm, symbol Connector:TestPoint
- R23: value 9.1K -> 10K
Connections:
- net 5V is gone; now on net +5V: J3.2 (Pin_2)
- net ADC0: now also J4.7 (Pin_7)
- net ADC2: now also J4.9 (Pin_9); no longer J4.10 (Pin_10)
- net ADC3: now also J4.10 (Pin_10); no longer J3.9 (Pin_9)
- net GND: now also J5.8 (Pin_8), J5.9 (Pin_9); no longer J3.10 (Pin_10)
- net GPIO17: now also J3.6 (Pin_6); no longer J5.7 (Pin_7)
- net GPIO6: now also J3.9 (Pin_9); no longer J5.1 (Pin_1)
- net GPIO7: now also J3.8 (Pin_8); no longer J5.2 (Pin_2)
- net GPIO8: now also J3.10 (Pin_10); no longer J5.3 (Pin_3)
- net I2C1_SCL: now also J5.4 (Pin_4); no longer J4.4 (Pin_4)
- net I2C1_SDA: now also J5.3 (Pin_3); no longer J4.3 (Pin_3)
- net LED_Data_Out: now also J5.7 (Pin_7); no longer J4.5 (Pin_5)
- net SPI0_RX: now also J3.7 (Pin_7); no longer J5.6 (Pin_6)
- net SPI0_SCK: now also J3.5 (Pin_5); no longer J5.8 (Pin_8)
- net SPI0_TX: now also J3.4 (Pin_4); no longer J5.9 (Pin_9)
- net UART0_RX: now also J5.5 (Pin_5)
- net UART0_TX: now also J5.6 (Pin_6); no longer TP6.1
- net UART1_RX: now also J5.1 (Pin_1); no longer J4.7 (Pin_7)
- net UART1_TX: now also J5.2 (Pin_2); no longer J4.6 (Pin_6)
- net VBUS: now also TP6.1
- net at J4.8 (Pin_8): now also R19.2
- net CAN_CS renamed GPIO24
- net GPIO24: now also J4.5 (Pin_5)
- net CAN_INT0 renamed GPIO22
- net GPIO22: now also J4.3 (Pin_3)
- net CAN_INT1 renamed GPIO23
- net GPIO23: now also J4.4 (Pin_4)
- net PWM_COB renamed GPIO25
- net GPIO25: now also J4.6 (Pin_6)
- removed net RS232_TX: J5.4 (Pin_4), J5.5 (Pin_5)
Other:
- moved on the sheet: C39, C40
