File: Electronic/Astronaut/core1106.kicad_sch (KiCad schematic)
At the start: 7 parts, among them J9 TC2050, U9 Core1106

Commit message: WIP Astronaut : completed most of the routing / schematic : next audio / power protection
Parts:
- removed TP5, TP6: TestPoint, symbol Connector:TestPoint
- added JP4: Jumper_3_Open, Jumper:SolderJumper-3_P1.3mm_Open_RoundedPad1.0x1.5mm_NumberLabels, symbol Jumper:Jumper_3_Open
- added JP5: Jumper_2_Open, Jumper:SolderJumper-2_P1.3mm_Open_RoundedPad1.0x1.5mm, symbol Jumper:Jumper_2_Open
- added TP3: TestPoint, TestPoint:TestPoint_Pad_D1.5mm, symbol Connector:TestPoint
- TP4: renamed from TP7; footprint (none) -> TestPoint:TestPoint_Pad_D1.5mm
- TP5: renamed from TP8; footprint (none) -> TestPoint:TestPoint_Pad_D1.5mm
- renumbered C25 to C31, J9 to J4
Connections:
- net +3.3V: now also J4.1, JP5.2 (B); no longer U9.78 (VCC_3V3)
- net +5V: now also JP4.1 (A)
- net BOOT: now also J4.9
- net GND: now also J4.3, JP4.3 (B)
- net GPIO3_A6: now also J4.2
- net GPIO3_A7: now also J4.4
- net RESET: now also J4.10
- net at J4.5: now also JP4.2 (C)
- net JTAG_MCU_TCK: now reaches J4.7
- net JTAG_MCU_TCK: now also U9.72 (JTAG_CPU_TCK_M1/UART2_TX_M1/JTAG_HPMCU_TCK_M0/JTAG_LPMCU_TCK_M0/GPIO1_B2_d)
- net JTAG_MCU_TMS: now reaches J4.8
- net JTAG_MCU_TMS: now also U9.73 (JTAG_CPU_TMS_M1/UART2_RX_M1/JTAG_HPMCU_TMS_M0/JTAG_LPMCU_TMS_M0/GPIO1_B3_u)
- net at U9.24 (USB_VBUSDET): now also TP3.1
- net ADC1: no longer names the net of U9.27 (SARADC_IN1/PWM1_M1/GPIO4_C1_z)
- new net: JP5.1 (A), U9.78 (VCC_3V3)
- no-connect marks 4 -> 33
Other:
- moved on the sheet: J4
